Commit message: generated a new urdf

File: fanuc_m20ib25_description/urdf/fanuc_m20ib25.urdf (robot description, URDF)
Before this commit: robot m-20ib25, 7 links, 6 joints
Links:
- link M-20iB25_axis1_1: geometry collision mesh filename=package://fanuc_m20ib25_description/meshes/M-20iB25_axis1_1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 scale=0.001 0.001 0.001; visual mesh filename=package://fanuc_m20ib25_description/meshes/M-20iB25_axis1_1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 scale=0.001 0.001 0.001
- link M-20iB25_axis2_1: geometry collision mesh filename=package://fanuc_m20ib25_description/meshes/M-20iB25_axis2_1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 scale=0.001 0.001 0.001; visual mesh filename=package://fanuc_m20ib25_description/meshes/M-20iB25_axis2_1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 scale=0.001 0.001 0.001
- link M-20iB25_axis3_1: geometry collision mesh filename=package://fanuc_m20ib25_description/meshes/M-20iB25_axis3_1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 scale=0.001 0.001 0.001; visual mesh filename=package://fanuc_m20ib25_description/meshes/M-20iB25_axis3_1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 scale=0.001 0.001 0.001
- link M-20iB25_axis4_1: geometry collision mesh filename=package://fanuc_m20ib25_description/meshes/M-20iB25_axis4_1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 scale=0.001 0.001 0.001; visual mesh filename=package://fanuc_m20ib25_description/meshes/M-20iB25_axis4_1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 scale=0.001 0.001 0.001
- link M-20iB25_axis5_1: geometry collision mesh filename=package://fanuc_m20ib25_description/meshes/M-20iB25_axis5_1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 scale=0.001 0.001 0.001; visual mesh filename=package://fanuc_m20ib25_description/meshes/M-20iB25_axis5_1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 scale=0.001 0.001 0.001
- link M-20iB25_axis6_1: geometry collision mesh filename=package://fanuc_m20ib25_description/meshes/M-20iB25_axis6_1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 scale=0.001 0.001 0.001; visual mesh filename=package://fanuc_m20ib25_description/meshes/M-20iB25_axis6_1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 scale=0.001 0.001 0.001
- link base_link: geometry collision mesh filename=package://fanuc_m20ib25_description/meshes/base_link.stl scale=0.001 0.001 0.001; visual mesh filename=package://fanuc_m20ib25_description/meshes/base_link.stl scale=0.001 0.001 0.001
